File: Fans.kicad_sch (KiCad schematic)
At the start: 12 parts, among them J2 Conn_01x03, J6 Conn_01x03, Q1 NMOS, Q3 NMOS

Commit message: Added pull up resistors for open drain configs
Parts:
- D1: renamed from D3; footprint Diode_SMD:D_SOD-123 -> Diode_SMD:D_SOD-323
- D2: renamed from D1; footprint Diode_SMD:D_SOD-123 -> Diode_SMD:D_SOD-323
- renumbered J6 to J2, J2 to J3, Q3 to Q1, Q1 to Q2, R10 to R4, R1 to R5, R16 to R6, R19 to R7, R5 to R8, R6 to R9

Commit message: Initial schematic design with 2 temp, 1 flow, 1 pump
Parts:
- renumbered D2 to D1, D1 to D2, J3 to FAN1, J2 to FAN2, Q2 to Q1, Q1 to Q2, R4 to R10, R8 to R5, R9 to R6, R5 to R7, R6 to R8, R7 to R9
