File: FlowrateSensor.kicad_sch (KiCad schematic)
At the start: 3 parts, among them J4 Conn_01x03

Commit message: Added pull up resistors for open drain configs
Parts:
- renumbered J4 to J7, R8 to R16, R9 to R17
Changed lines of the file:
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@@
 		(on_board yes)
 		(dnp no)
-		(property "Reference" "R9"
+		(property "Reference" "R17"
 			(at 91.44 55.8799 0)
 			(effects
@@
 			(project "PTN-PumpControlBoard"
 				(path "/591f46f8-eb1d-42dc-a4cb-8182eac4ef58/72cbb232-97a0-4b9b-a6b0-3f04462a78a5"
-					(reference "R9")
+					(reference "R17")
 					(unit 1)
 				)
@@
 		(dnp no)
 		(fields_autoplaced yes)
-		(property "Reference" "J4"
+		(property "Reference" "J7"
 			(at 64.77 49.5299 0)
 			(effects
@@
 			(project "PTN-PumpControlBoard"
 				(path "/591f46f8-eb1d-42dc-a4cb-8182eac4ef58/72cbb232-97a0-4b9b-a6b0-3f04462a78a5"
-					(reference "J4")
+					(reference "J7")
 					(unit 1)
 				)
@@
 		(dnp no)
 		(fields_autoplaced yes)
-		(property "Reference" "#PWR08"
+		(property "Reference" "#PWR037"
 			(at 52.07 64.77 0)
 			(effects
@@
 			(project "PTN-PumpControlBoard"
 				(path "/591f46f8-eb1d-42dc-a4cb-8182eac4ef58/72cbb232-97a0-4b9b-a6b0-3f04462a78a5"
-					(reference "#PWR08")
+					(reference "#PWR037")
 					(unit 1)
 				)
@@
 		(on_board yes)
 		(dnp no)
-		(property "Reference" "R8"
+		(property "Reference" "R16"
 			(at 91.44 43.1799 0)
 			(effects
@@
 			(project "PTN-PumpControlBoard"
 				(path "/591f46f8-eb1d-42dc-a4cb-8182eac4ef58/72cbb232-97a0-4b9b-a6b0-3f04462a78a5"
-					(reference "R8")
+					(reference "R16")
 					(unit 1)
 				)
@@
 		(dnp no)
 		(fields_autoplaced yes)
-		(property "Reference" "#PWR033"
+		(property "Reference" "#PWR038"
 			(at 88.9 69.85 0)
 			(effects
@@
 			(project "PTN-PumpControlBoard"
 				(path "/591f46f8-eb1d-42dc-a4cb-8182eac4ef58/72cbb232-97a0-4b9b-a6b0-3f04462a78a5"
-					(reference "#PWR033")
-					(unit 1)
-				)
+					(reference "#PWR038")
+					(unit 1)
+				)

Commit message: Initial schematic design with 2 temp, 1 flow, 1 pump
Parts:
- removed R16: 10k, Resistor_SMD:R_0805_2012Metric, symbol Device:R_US
- removed R17: 3.8k, Resistor_SMD:R_0805_2012Metric, symbol Device:R_US
- added Q3: NMOS, Package_TO_SOT_SMD:LFPAK33, symbol Simulation_SPICE:NMOS
- added R19, R20: 10k, Resistor_SMD:R_0805_2012Metric, symbol Device:R_US
- renumbered J7 to FLOW1
Connections:
- net FLOW_OUT: now also Q3.2 (G), R19.1
- net FLOW_SEN: now also Q3.3 (S), R19.2, R20.1
- net GND: now also R20.2
- new net +3.3V: Q3.1 (D)
