File: PTN-PumpControlBoard.kicad_pcb (KiCad board)
At the start: 2 copper layers, 38 parts, among them IC1 ADT7470ARQZ-REEL7, J1 Conn_01x04, J2 Conn_01x03, J3 Conn_01x02, J4 Conn_01x03, J5 Conn_01x04, J6 Conn_01x02, J7 Conn_01x03, Q1 NMOS, Q2 NMOS, SW1 SW_Push, SW2 SW_Push, SW3 SW_Push, U1 PeripheralSOM, U2 ADS130B02QPWRQ1, U3 ST7735R

Commit message: Added pull up resistors for open drain configs
Parts:
- removed D2: 1N4448W, Diode_SMD:D_SOD-123
- removed J7: Conn_01x03, UTSVT_Connectors:Molex_MicroFit3.0_1x3xP3.00mm_PolarizingPeg_Vertical
- removed Q2: NMOS, Package_TO_SOT_SMD:LFPAK33
- removed R12: 1k, Resistor_SMD:R_0805_2012Metric
- removed R13: 380, Resistor_SMD:R_0805_2012Metric
- removed U2: ADS130B02QPWRQ1, ADC:TSSOP20_PW_TEX
- added C6: 10n, Capacitor_SMD:C_0805_2012Metric, F.Cu at (238.6, 56.9)
- added D3: 1N4448W, Diode_SMD:D_SOD-323, F.Cu at (253.9, 53.5)
- added IC2: ADS131M03QPWRQ1, ADC2:SOP65P640X120-20N, F.Cu at (240.8, 51.3)
- added J10: Conn_01x02, UTSVT_Connectors:Molex_MicroFit3.0_1x2xP3.00mm_PolarizingPeg_Vertical, F.Cu at (241.5, 41.5)
- added J9: Conn_01x02, UTSVT_Connectors:Molex_MicroFit3.0_1x2xP3.00mm_PolarizingPeg_Vertical, F.Cu at (241.5, 34.3)
- added Q3: NMOS, Package_TO_SOT_SMD:LFPAK33, F.Cu at (254.4, 49.6)
- added R16: 1k, Resistor_SMD:R_0805_2012Metric, F.Cu at (249.5, 48.7)
- added R17: 3.5k, Resistor_SMD:R_0805_2012Metric, F.Cu at (251.7, 32.2)
- added R18: 3.5k, Resistor_SMD:R_0805_2012Metric, F.Cu at (251.7, 35.1)
- added R19: 380, Resistor_SMD:R_0805_2012Metric, F.Cu at (249.5, 51.6)
- D1: footprint Diode_SMD:D_SOD-123 -> Diode_SMD:D_SOD-323
- J6: value Conn_01x02 -> Conn_01x03; footprint UTSVT_Connectors:Molex_MicroFit3.0_1x2xP3.00mm_PolarizingPeg_Vertical -> UTSVT_Connectors:Molex_MicroFit3.0_1x3xP3.00mm_PolarizingPeg_Vertical
- R10: value 3.5k -> 10k
Connections:
- net /FLOW_SEN renamed /FLOW
- net /Fan1/TACH1_IN renamed /Fans/TACH1_IN
- net /TEMP_SEN1 renamed /TEMP1
- C5 pad 2: /TEMP_SEN2 -> /TEMP2
- J6 pad 1: GND -> +12V
- J6 pad 2: /TEMP_SEN2 -> /Fans/TACH2_IN
- R10 pad 1: +3.3V -> /FAN2_PWM
- R10 pad 2: /TEMP_SEN2 -> GND
- R11 pad 1: /FAN2_PWM -> /~{SMBALERT}
- R11 pad 2: GND -> +3.3V

Commit message: Initial schematic design with 2 temp, 1 flow, 1 pump
Parts:
- removed C6: 10n, Capacitor_SMD:C_0805_2012Metric
- removed D3: 1N4448W, Diode_SMD:D_SOD-323
- removed IC1: ADT7470ARQZ-REEL7, Package_SO:QSOP-16_3.9x4.9mm_P0.635mm
- removed IC2: ADS131M03QPWRQ1, ADC2:SOP65P640X120-20N
- removed J10, J3, J9: Conn_01x02, UTSVT_Connectors:Molex_MicroFit3.0_1x2xP3.00mm_PolarizingPeg_Vertical
- removed J2, J4, J6: Conn_01x03, UTSVT_Connectors:Molex_MicroFit3.0_1x3xP3.00mm_PolarizingPeg_Vertical
- removed J5: Conn_01x04, UTSVT_Connectors:Molex_MicroFit3.0_1x4xP3.00mm_PolarizingPeg_Vertical
- added D2: 1N4448W, Diode_SMD:D_SOD-323, F.Cu at (113.4, 118.0)
- added FAN1: Conn_01x03, UTSVT_Connectors:Molex_MicroFit3.0_1x3xP3.00mm_PolarizingPeg_Vertical, F.Cu at (109.2, 110.0)
- added FAN2: Conn_01x03, UTSVT_Connectors:Molex_MicroFit3.0_1x3xP3.00mm_PolarizingPeg_Vertical, F.Cu at (109.2, 126.9)
- added FLOW1: Conn_01x03, UTSVT_Connectors:Molex_MicroFit3.0_1x3xP3.00mm_PolarizingPeg_Vertical, F.Cu at (155.1, 130.2)
- added PUMP1: Conn_01x04, UTSVT_Connectors:Molex_MicroFit3.0_1x4xP3.00mm_PolarizingPeg_Vertical, F.Cu at (109.2, 93.0)
- added Q2: NMOS, Package_TO_SOT_SMD:LFPAK33, F.Cu at (116.5, 118.1)
- added R12: 1k, Resistor_SMD:R_0805_2012Metric, F.Cu at (180.9, 126.8)
- added R13: 1k, Resistor_SMD:R_0805_2012Metric, F.Cu at (192.5, 126.8)
- added R20: 10k, Resistor_SMD:R_0805_2012Metric, F.Cu at (149.1, 126.3)
- added TEMP1: Conn_01x02, UTSVT_Connectors:Molex_MicroFit3.0_1x2xP3.00mm_PolarizingPeg_Vertical, F.Cu at (117.9, 69.6)
- added TEMP2: Conn_01x02, UTSVT_Connectors:Molex_MicroFit3.0_1x2xP3.00mm_PolarizingPeg_Vertical, F.Cu at (132.8, 69.6)
- added U2: PeripheralSOM, UTSVT_Special:PeripheralSOM, F.Cu at (145.7, 105.0)
- C2: value 220n -> 1uF
- C3: value 1uF -> 0.1uF
- C4: value 10n -> 0.1uF
- C5: value 50n -> 0.1uF
- J1: value Conn_01x04 -> PeripheralCANConnector
- R11, R8: value 10k -> 1k
- R16: value 1k -> 10k
- R17, R18: value 3.5k -> 1k
- R19: value 380 -> 10k
- R4: value 10k -> 15k
- R7: value 3.5k -> 10k
- R9: value 3.8k -> 380
- U1: value PeripheralSOM -> EMC2305-1-AP-TR; footprint UTSVT_Special:PeripheralSOM -> FanControl:QFN16_4x4MC_MCH
- moved R17 135.3 mm to (123.0, 74.0), turned to 180 degrees
- moved Q3 125.9 mm to (152.3, 123.2), turned to -90 degrees
- moved U1 125.3 mm to (125.0, 113.2), turned to -90 degrees
- moved R19 120.0 mm to (155.5, 126.2), turned to 90 degrees
- moved R18 119.9 mm to (138.2, 73.6), turned to 180 degrees
- moved R7 117.0 mm to (120.5, 109.4), turned to 180 degrees
- moved R10 116.6 mm to (120.1, 118.8), turned to 180 degrees
- moved C2 103.1 mm to (128.8, 115.6), turned to 90 degrees
- moved C1 102.7 mm to (128.8, 112.0), turned to 90 degrees
- moved R16 94.6 mm to (196.1, 126.8)
- moved D1 93.8 mm to (113.7, 109.0), turned to 90 degrees
- moved R14 92.3 mm to (172.6, 126.6)
- moved Q1 89.2 mm to (116.7, 108.4), turned to 90 degrees
- moved R5 87.4 mm to (116.7, 114.4)
- moved R6 85.4 mm to (116.7, 112.4), turned to 180 degrees
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Connections:
- C2 pad 1: DGND -> +3.3V
- C2 pad 2: Net-(IC2-CAP) -> GND
- C3 pad 1: Net-(IC2-AVDD) -> GND
- C3 pad 2: AGND -> /FAN_SPEED
- C4 pad 1: /TEMP1 -> GND
- C4 pad 2: Net-(IC2-AIN0N) -> /PUMP_SPEED
- C5 pad 1: Net-(IC2-AIN1N) -> GND
- C5 pad 2: /TEMP2 -> /SYST_MODE
- Q3 pad 1: Net-(D3-A) -> +3.3V
- Q3 pad 2: /FAN2_PWM -> /FlowrateSensor/FLOW_OUT
- Q3 pad 3: GND -> /FLOW
- R1 pad 1: /FAN1_PWM -> /~{SMBALERT}
- R1 pad 2: GND -> +3.3V
- R11 pad 1: /~{SMBALERT} -> Net-(R11-Pad1)
- R11 pad 2: +3.3V -> /FAN_SPEED
- R14 pad 1: +3.3V -> Net-(R11-Pad1)
- R14 pad 2: /FAN2_PWM -> GND
- R15 pad 1: /FAN1_PWM -> Net-(R12-Pad1)
- R15 pad 2: +3.3V -> GND
- R16 pad 1: /Fans/TACH2_IN -> Net-(R13-Pad1)
- R16 pad 2: /FAN2_TACH -> GND
- R17 pad 1: +12V -> +3.3V
- R17 pad 2: /TEMP2 -> /TEMP1
- R18 pad 1: +12V -> +3V3
- R18 pad 2: /TEMP3 -> /TEMP2
- R19 pad 1: /FAN2_TACH -> /FlowrateSensor/FLOW_OUT
- R19 pad 2: GND -> /FLOW
- R2 pad 1: /FAN_SPEED -> /FAN2_PWM
- R2 pad 2: GND -> +3.3V
- R3 pad 1: /PUMP_SPEED -> /FAN1_PWM
- R3 pad 2: GND -> +3.3V
- R4 pad 1: /SYST_MODE -> Net-(U1-CLK)
- R4 pad 2: GND -> +3.3V
- R7 pad 1: +12V -> /FAN1_PWM
- R7 pad 2: /TEMP1 -> GND
- R8 pad 1: /FlowrateSensor/FLOW_OUT -> /Fans/TACH2_IN
- R8 pad 2: /FLOW -> /FAN2_TACH
- R9 pad 1: /FLOW -> /FAN2_TACH
- SW1 pad 1: /FAN_SPEED -> Net-(R11-Pad1)
- SW2 pad 1: /PUMP_SPEED -> Net-(R12-Pad1)
- SW3 pad 1: /SYST_MODE -> Net-(R13-Pad1)
- U1 pad 1: /MOSI -> /FAN_SCL
- U1 pad 10: +3.3V -> unconnected-(U1-TACH3-Pad10)
- U1 pad 11: DGND -> Net-(U1-CLK)
- U1 pad 12: AGND -> /~{SMBALERT}
- U1 pad 13: /~{SMBALERT} -> unconnected-(U1-PWM4-Pad13)
- U1 pad 14: /SYST_MODE -> unconnected-(U1-TACH4-Pad14)
- U1 pad 15: /~{DRDY} -> unconnected-(U1-PWM5-Pad15)
- U1 pad 16: /FLOW -> unconnected-(U1-TACH5-Pad16)
- U1 pad 2: +3.3V -> /FAN_SDA
- U1 pad 3: /MISO -> +3.3V
- U1 pad 4: GND -> unconnected-(U1-ADDR_SEL-Pad4)
- U1 pad 5: /SCLK -> /FAN1_PWM
- U1 pad 6: /FAN_SDA -> /FAN1_TACH
- U1 pad 7: /ADC_~{CS} -> /FAN2_PWM
- U1 pad 8: /FAN_SCL -> /FAN2_TACH
- U1 pad 9: +3.3V -> unconnected-(U1-PWM3-Pad9)
Routing:
- net /SYST_MODE: track 0.00 -> 76.0 mm
- net /LCD_TFT_~{CS}: track 0.00 -> 71.5 mm
- net /SCLK: track 0.00 -> 70.3 mm
- net /MOSI: track 0.00 -> 64.7 mm
- net /PUMP_SPEED: track 0.00 -> 63.2 mm
- net /LCD_RESET: track 0.00 -> 54.2 mm
- net /FAN_SPEED: track 0.00 -> 49.8 mm
- net /FLOW: track 0.00 -> 43.1 mm
- net CAN_L: track 0.00 -> 40.8 mm
- net GNDPWR: track 0.00 -> 38.6 mm
- net CAN_H: track 0.00 -> 38.1 mm
- net /TEMP2: track 0.00 -> 36.6 mm
- net /TEMP1: track 0.00 -> 32.6 mm
- net /PUMP_PWM: track 0.00 -> 20.5 mm
- net /PUMP_PG: track 0.00 -> 19.5 mm
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- added copper zone on F.Cu, net +12V
- added copper zone on F.Cu, net +3.3V
- added copper zone on B.Cu, net GND
Other:
- board outline added: 100.2 x 72 mm
