File: Pump.kicad_sch (KiCad schematic)
At the start: 1 part, among them J5 Conn_01x04

Commit message: Added pull up resistors for open drain configs
Parts:
- renumbered J5 to J8
Changed lines of the file:
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@@
 		(dnp no)
 		(fields_autoplaced yes)
-		(property "Reference" "#PWR032"
+		(property "Reference" "#PWR039"
 			(at 41.91 48.26 0)
 			(effects
@@
 			(project "PTN-PumpControlBoard"
 				(path "/591f46f8-eb1d-42dc-a4cb-8182eac4ef58/49b28e86-cfde-410d-931b-2f924e16f8d9"
-					(reference "#PWR032")
+					(reference "#PWR039")
 					(unit 1)
 				)
@@
 		(dnp no)
 		(fields_autoplaced yes)
-		(property "Reference" "J5"
+		(property "Reference" "J8"
 			(at 52.07 35.5599 0)
 			(effects
@@
 			(project "PTN-PumpControlBoard"
 				(path "/591f46f8-eb1d-42dc-a4cb-8182eac4ef58/49b28e86-cfde-410d-931b-2f924e16f8d9"
-					(reference "J5")
+					(reference "J8")
 					(unit 1)
 				)

Commit message: Initial schematic design with 2 temp, 1 flow, 1 pump
Parts:
- renumbered J8 to PUMP1
Changed lines of the file:
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@@
 		(dnp no)
 		(fields_autoplaced yes)
-		(property "Reference" "#PWR039"
+		(property "Reference" "#PWR033"
 			(at 41.91 48.26 0)
 			(effects
@@
 			(project "PTN-PumpControlBoard"
 				(path "/591f46f8-eb1d-42dc-a4cb-8182eac4ef58/49b28e86-cfde-410d-931b-2f924e16f8d9"
-					(reference "#PWR039")
+					(reference "#PWR033")
 					(unit 1)
 				)
@@
 		(dnp no)
 		(fields_autoplaced yes)
-		(property "Reference" "J8"
+		(property "Reference" "PUMP1"
 			(at 52.07 35.5599 0)
 			(effects
@@
 			)
 		)
-		(property "Datasheet" "~"
+		(property "Datasheet" "https://freezemod.com/product/freezemod-computer-water-cooler-magnetic-levitation-domestic-ddc-water-pump-pub-gcdcb-pm/"
 			(at 49.53 35.56 0)
 			(effects
@@
 			(project "PTN-PumpControlBoard"
 				(path "/591f46f8-eb1d-42dc-a4cb-8182eac4ef58/49b28e86-cfde-410d-931b-2f924e16f8d9"
-					(reference "J8")
+					(reference "PUMP1")
 					(unit 1)
 				)
