File: Switches.kicad_sch (KiCad schematic)
At the start: 6 parts, among them SW1 SW_Push, SW2 SW_Push, SW3 SW_Push

Commit message: Added pull up resistors for open drain configs
Parts:
- renumbered R2 to R10, R3 to R11, R4 to R12
Changed lines of the file:
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@@
 		(dnp no)
 		(fields_autoplaced yes)
-		(property "Reference" "#PWR05"
+		(property "Reference" "#PWR028"
 			(at 72.39 71.12 0)
 			(effects
@@
 			(project "PTN-PumpControlBoard"
 				(path "/591f46f8-eb1d-42dc-a4cb-8182eac4ef58/1bf99de6-cde9-4f3c-86c0-48afb50edfd0"
-					(reference "#PWR05")
+					(reference "#PWR028")
 					(unit 1)
 				)
@@
 		(dnp no)
 		(fields_autoplaced yes)
-		(property "Reference" "#PWR014"
+		(property "Reference" "#PWR029"
 			(at 106.68 39.37 0)
 			(effects
@@
 			(project "PTN-PumpControlBoard"
 				(path "/591f46f8-eb1d-42dc-a4cb-8182eac4ef58/1bf99de6-cde9-4f3c-86c0-48afb50edfd0"
-					(reference "#PWR014")
+					(reference "#PWR029")
 					(unit 1)
 				)
@@
 		(on_board yes)
 		(dnp no)
-		(property "Reference" "R2"
+		(property "Reference" "R10"
 			(at 40.64 55.8799 0)
 			(effects
@@
 			(project "PTN-PumpControlBoard"
 				(path "/591f46f8-eb1d-42dc-a4cb-8182eac4ef58/1bf99de6-cde9-4f3c-86c0-48afb50edfd0"
-					(reference "R2")
+					(reference "R10")
 					(unit 1)
 				)
@@
 		(dnp no)
 		(fields_autoplaced yes)
-		(property "Reference" "#PWR015"
+		(property "Reference" "#PWR030"
 			(at 106.68 71.12 0)
 			(effects
@@
 			(project "PTN-PumpControlBoard"
 				(path "/591f46f8-eb1d-42dc-a4cb-8182eac4ef58/1bf99de6-cde9-4f3c-86c0-48afb50edfd0"
-					(reference "#PWR015")
+					(reference "#PWR030")
 					(unit 1)
 				)
@@
 		(dnp no)
 		(fields_autoplaced yes)
-		(property "Reference" "#PWR04"
+		(property "Reference" "#PWR027"
 			(at 72.39 39.37 0)
 			(effects
@@
 			(project "PTN-PumpControlBoard"
 				(path "/591f46f8-eb1d-42dc-a4cb-8182eac4ef58/1bf99de6-cde9-4f3c-86c0-48afb50edfd0"
-					(reference "#PWR04")
+					(reference "#PWR027")
 					(unit 1)
 				)
@@
 		(on_board yes)
 		(dnp no)
-		(property "Reference" "R4"
+		(property "Reference" "R12"
 			(at 109.22 55.8799 0)
 			(effects
@@
 			(project "PTN-PumpControlBoard"
 				(path "/591f46f8-eb1d-42dc-a4cb-8182eac4ef58/1bf99de6-cde9-4f3c-86c0-48afb50edfd0"
-					(reference "R4")
+					(reference "R12")
 					(unit 1)
 				)
@@
 		(dnp no)
 		(fields_autoplaced yes)
-		(property "Reference" "#PWR01"
+		(property "Reference" "#PWR025"
 			(at 38.1 39.37 0)
 			(effects
@@
 			(project "PTN-PumpControlBoard"
 				(path "/591f46f8-eb1d-42dc-a4cb-8182eac4ef58/1bf99de6-cde9-4f3c-86c0-48afb50edfd0"
-					(reference "#PWR01")
+					(reference "#PWR025")
 					(unit 1)
 				)
@@
 		(on_board yes)
 		(dnp no)
-		(property "Reference" "R3"
+		(property "Reference" "R11"
 			(at 74.93 55.8799 0)
 			(effects
@@
 			(project "PTN-PumpControlBoard"
 				(path "/591f46f8-eb1d-42dc-a4cb-8182eac4ef58/1bf99de6-cde9-4f3c-86c0-48afb50edfd0"
-					(reference "R3")
+					(reference "R11")
 					(unit 1)
 				)
@@
 		(dnp no)
 		(fields_autoplaced yes)
-		(property "Reference" "#PWR02"
+		(property "Reference" "#PWR026"
 			(at 38.1 71.12 0)
 			(effects
@@
 			(project "PTN-PumpControlBoard"
 				(path "/591f46f8-eb1d-42dc-a4cb-8182eac4ef58/1bf99de6-cde9-4f3c-86c0-48afb50edfd0"
-					(reference "#PWR02")
-					(unit 1)
-				)
+					(reference "#PWR026")
+					(unit 1)
+				)

Commit message: Initial schematic design with 2 temp, 1 flow, 1 pump
Parts:
- added C3, C4, C5: 0.1uF, Capacitor_SMD:C_0805_2012Metric, symbol Device:C
- added R11, R12, R13: 1k, Resistor_SMD:R_0805_2012Metric, symbol Device:R_US
- renumbered R10 to R14, R11 to R15, R12 to R16
Connections:
- net FAN_SPEED: now also C3.2, R11.2; no longer R14.1, SW1.1
- net GND: now also C3.1, C4.1, C5.1
- net PUMP_SPEED: now also C4.2, R12.2; no longer R15.1, SW2.1
- net SYST_MODE: now also C5.2, R13.2; no longer R16.1, SW3.1
- new net: R12.1, R15.1, SW2.1
- new net: R11.1, R14.1, SW1.1
- new net: R13.1, R16.1, SW3.1
Other:
- moved on the sheet: R15, R16, SW2, SW3
